File: Max50x100Plate.kicad_pcb (KiCad board)
At the start: 2 copper layers, 100 x 50 mm, 6 parts

Commit message: JLC Design Rules
Save as KiCad 7.
Set design rules to JLCPCB 2-layer capabilities.
Other:
- board text added: "MaxPlate 50x100 Copyright Andrew Fischer 2023 CC BY-NC-4.0 24032023"
- board text removed: "MaxPlate 50x100 Copyright Andrew Fischer 2023 CC-BY-NC-4.0 23012023"
